File: PlatineA_CNMB2/PlatineA_CNMB2.kicad_pcb (KiCad board)
At the start: 2 copper layers, 86.5 x 33 mm, 34 parts, among them IC1 MC34063AD, IC2 MAX487E, IC3 ATmega328P-A, J1 Nano_Conn, J2 Screw_Terminal_01x06, J3 RS485_Conn, J4 24V_Terminal, J5 BUS_Terminal, J6 AVR-ISP-6, Y1 16Mhz

Commit message: Add files via upload
Connections:
- IC3 pad 13: /1WIRE -> /D9
- IC3 pad 14: /D10 -> /1WIRE
Changed lines of the file:
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@@
 			(size 1.6 0.55)
 			(layers "B.Cu" "B.Mask" "B.Paste")
-			(net "/1WIRE")
+			(net "/D9")
 			(pinfunction "PB1_13")
 			(pintype "bidirectional")
@@
 			(size 1.6 0.55)
 			(layers "B.Cu" "B.Mask" "B.Paste")
-			(net "/D10")
+			(net "/1WIRE")
 			(pinfunction "PB2_14")
 			(pintype "bidirectional")
@@
 	)
 	(segment
-		(start 142.02 102.28)
-		(end 143.12 101.18)
+		(start 178.044544 91.8)
+		(end 183.624544 97.38)
 		(width 0.3)
 		(layer "B.Cu")
@@
 	)
 	(segment
-		(start 178.044544 91.8)
-		(end 183.624544 97.38)
+		(start 187.65 110.77)
+		(end 185.8 112.62)
 		(width 0.3)
 		(layer "B.Cu")
@@
 	)
 	(segment
-		(start 142.02 103.38)
-		(end 142.02 102.28)
+		(start 143.12 96.287057)
+		(end 146.05 93.357057)
 		(width 0.3)
 		(layer "B.Cu")
@@
 	)
 	(segment
-		(start 187.65 110.77)
-		(end 185.8 112.62)
+		(start 142.82 101.48)
+		(end 142.82 103.38)
 		(width 0.3)
 		(layer "B.Cu")
@@
 	)
 	(segment
-		(start 143.12 96.287057)
-		(end 146.05 93.357057)
+		(start 143.12 101.18)
+		(end 142.82 101.48)
 		(width 0.3)
 		(layer "B.Cu")
