File: PlatineA_CNMB2/PlatineA_CNMB2.kicad_sch (KiCad schematic)
At the start: 34 parts, among them IC1 MC34063AD, IC2 MAX487E, IC3 ATmega328P-A, J1 Nano_Conn, J2 Screw_Terminal_01x06, J3 RS485_Conn, J4 24V_Terminal, J5 BUS_Terminal, J6 AVR-ISP-6, Y1 16Mhz

Commit message: Add files via upload
Connections:
- net D10 is gone; now on net 1WIRE: IC3.14 (PB2)
- net 1WIRE: no longer IC3.13 (PB1)
- new net D9: IC3.13 (PB1)
Changed lines of the file:
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@@
+	(wire
+		(pts
+			(xy 78.232 98.552) (xy 78.232 104.902)
+		)
+		(stroke
+			(width 0)
+			(type default)
+		)
+	)
 	(wire
 		(pts
@@
 	(wire
 		(pts
-			(xy 78.232 98.552) (xy 78.232 102.362)
-		)
-		(stroke
-			(width 0)
-			(type default)
-		)
-	)
-	(wire
-		(pts
 			(xy 58.166 89.916) (xy 60.706 89.916)
 		)
@@
 	(wire
 		(pts
-			(xy 78.232 102.362) (xy 73.406 102.362)
-		)
-		(stroke
+			(xy 78.232 104.902) (xy 73.406 104.902)
+		)
+		(stroke
